Commit message: mount arm into correct position

File: cob_hardware_config/robots/p_rob/urdf/p_rob.urdf.xacro (robot description, xacro)
@@ -38,5 +38,5 @@
   </xacro:raw_head>
   <xacro:p_rob name="arm" parent="base_link">
-    <origin xyz="${arm_x} ${arm_y} ${arm_z}" rpy="${arm_roll} ${arm_pitch} ${arm_yaw}" />
+    <origin xyz="${arm_x} ${arm_y} ${arm_z}" rpy="${arm_roll} ${arm_pitch} ${arm_yaw+20}" />
   </xacro:p_rob>
 </robot>
