Commit message: correct camera clibration

File: cob_hardware_config/robots/cob4-10/urdf/calibration_default.urdf.xacro (robot description, xacro)
@@ -110,6 +110,6 @@
 	<xacro:property name="def_sensorring_cam3d_front_yaw" value="0.0"/>
 	<!-- cam3d | handeye calibration | relative to sensorring_link -->
-	<xacro:property name="def_sensorring_cam3d_back_x" value="-0.121"/>
-	<xacro:property name="def_sensorring_cam3d_back_y" value="-0.095"/>
+	<xacro:property name="def_sensorring_cam3d_back_x" value="-0.111"/>
+	<xacro:property name="def_sensorring_cam3d_back_y" value="-0.155"/>
 	<xacro:property name="def_sensorring_cam3d_back_z" value="0.0293"/>
 	<xacro:property name="def_sensorring_cam3d_back_roll" value="0.0"/>
