Commit message: testing kinova arm into cob

File: cob_hardware_config/robots/cob4-10/urdf/cob4-10.urdf.xacro (robot description, xacro)
@@ -13,4 +13,5 @@
   <!-- arm -->
   <xacro:include filename="$(find cob_description)/urdf/cob4_arm/cob4_arm.urdf.xacro" />
+  <xacro:include filename="$(find kinova_description)/urdf/j2n4s300.xacro"/>
   <!-- hand -->
   <xacro:include filename="$(find cob_description)/urdf/cob4_gripper/gripper.urdf.xacro" />
@@ -71,12 +72,7 @@
     <origin xyz="${arm_right_x} ${arm_right_y} ${arm_right_z}" rpy="${arm_right_roll} ${arm_right_pitch} ${arm_right_yaw}" />
   </xacro:cob4_arm>
-  <xacro:cob4_arm name="arm_left" parent="torso_3_link" has_podest="false">
+  <xacro:j2n4s300  base_parent="torso_3_link"/>
+  <!--xacro:cob4_arm name="arm_left" parent="torso_3_link" has_podest="false">
     <origin xyz="${arm_left_x} ${arm_left_y} ${arm_left_z}" rpy="${arm_left_roll} ${arm_left_pitch} ${arm_left_yaw}" />
-  </xacro:cob4_arm>
-  <xacro:gripper name="gripper_right" parent="arm_right_7_link">
-    <origin xyz="${gripper_right_x} ${gripper_right_y} ${gripper_right_z}" rpy="${gripper_right_roll} ${gripper_right_pitch} ${gripper_right_yaw}" />
-  </xacro:gripper>
-  <xacro:gripper name="gripper_left" parent="arm_left_7_link">
-    <origin xyz="${gripper_left_x} ${gripper_left_y} ${gripper_left_z}" rpy="${gripper_left_roll} ${gripper_left_pitch} ${gripper_left_yaw}" />
-  </xacro:gripper>
+  </xacro:cob4_arm-->
 </robot>

Commit message: config for fp_arm on cob4-10

File: cob_hardware_config/robots/cob4-10/urdf/cob4-10.urdf.xacro (robot description, xacro)
@@ -13,4 +13,6 @@
   <!-- arm -->
   <xacro:include filename="$(find cob_description)/urdf/cob4_arm/cob4_arm.urdf.xacro" />
+  <!-- p_rob_arm -->
+  <xacro:include filename="$(find cob_description)/urdf/p_rob/p_rob.urdf.xacro" />
   <!-- hand -->
   <xacro:include filename="$(find cob_description)/urdf/cob4_gripper/gripper.urdf.xacro" />
@@ -71,12 +73,9 @@
     <origin xyz="${arm_right_x} ${arm_right_y} ${arm_right_z}" rpy="${arm_right_roll} ${arm_right_pitch} ${arm_right_yaw}" />
   </xacro:cob4_arm>
-  <xacro:cob4_arm name="arm_left" parent="torso_3_link" has_podest="false">
+  <xacro:p_rob name="arm_left" parent="torso_3_link">
     <origin xyz="${arm_left_x} ${arm_left_y} ${arm_left_z}" rpy="${arm_left_roll} ${arm_left_pitch} ${arm_left_yaw}" />
-  </xacro:cob4_arm>
-  <xacro:gripper name="gripper_right" parent="arm_right_7_link">
-    <origin xyz="${gripper_right_x} ${gripper_right_y} ${gripper_right_z}" rpy="${gripper_right_roll} ${gripper_right_pitch} ${gripper_right_yaw}" />
-  </xacro:gripper>
-  <xacro:gripper name="gripper_left" parent="arm_left_7_link">
-    <origin xyz="${gripper_left_x} ${gripper_left_y} ${gripper_left_z}" rpy="${gripper_left_roll} ${gripper_left_pitch} ${gripper_left_yaw}" />
-  </xacro:gripper>
+  </xacro:p_rob>
+  <!--xacro:cob4_arm name="arm_left" parent="torso_3_link" has_podest="false">
+    <origin xyz="${arm_left_x} ${arm_left_y} ${arm_left_z}" rpy="${arm_left_roll} ${arm_left_pitch} ${arm_left_yaw}" />
+  </xacro:cob4_arm-->
 </robot>

File: cob_hardware_config/robots/raw3-1/urdf/raw3-1.urdf.xacro (robot description, xacro)
@@ -10,14 +10,8 @@
   <!-- raw tower -->
   <xacro:include filename="$(find raw_description)/urdf/tower_asymetric/tower.urdf.xacro" />
-  <!-- torso -->
-  <xacro:include filename="$(find raw_description)/urdf/torso/torso_v2.urdf.xacro" />
   <!-- p_rob_arm -->
-  <xacro:include filename="$(find raw_description)/urdf/p_rob_arm/p_rob.urdf.xacro" />
+  <xacro:include filename="$(find cob_description)/urdf/p_rob/p_rob.urdf.xacro" />
   <!-- vacuum gripper -->
   <!--xacro:include filename="$(find raw_description)/urdf/vacuum_gripper/gripper.urdf.xacro" /-->
-  <!-- schmaltz vacuum gripper -->
-  <xacro:include filename="$(find raw_description)/urdf/schmaltz_gripper/gripper.urdf.xacro" />
-  <!-- arm camera -->
-  <xacro:include filename="$(find raw_description)/urdf/kinect_camera/kinect_camera.urdf.xacro" />
   <!-- sensors -->
   <xacro:include filename="$(find cob_description)/urdf/sensors/sick_s300_laser.urdf.xacro"/>
@@ -35,12 +29,12 @@
     <origin xyz="${tower_x} ${tower_y} ${tower_z}" rpy="${tower_roll} ${tower_pitch} ${tower_yaw}" />
   </xacro:tower_asymetric>
-  <xacro:raw_torso_v2 name="torso" parent="base_link">
+  <!--xacro:raw_torso_v2 name="torso" parent="base_link">
     <origin xyz="${torso_x} ${torso_y} ${torso_z}" rpy="${torso_roll} ${torso_pitch} ${torso_yaw}" />
-  </xacro:raw_torso_v2>
+  </xacro:raw_torso_v2-->
   <xacro:p_rob name="arm" parent="base_link">
     <origin xyz="${arm_x} ${arm_y} ${arm_z}" rpy="${arm_roll} ${arm_pitch} ${arm_yaw - 3.49066}" />
   </xacro:p_rob>
-  <xacro:kinect_camera name="arm_camera" ros_topic="arm_kinect_camera" parent="gripper_coupling_link" update_rate="30" data_skip="9">
+  <!--xacro:kinect_camera name="arm_camera" ros_topic="arm_kinect_camera" parent="gripper_coupling_link" update_rate="30" data_skip="9">
     <origin xyz="${arm_camera_x} ${arm_camera_y} ${arm_camera_z}" rpy="${arm_camera_roll} ${arm_camera_pitch} ${arm_camera_yaw}" />
-  </xacro:kinect_camera>
+  </xacro:kinect_camera-->
 </robot>
