Commit message: merge with actual indigo dev+

File: cob_hardware_config/robots/raw3-1/urdf/calibration_default.urdf.xacro (robot description, xacro)
@@ -32,7 +32,7 @@
 	<xacro:property name="def_torso_y" value="0.2175"/>
 	<xacro:property name="def_torso_z" value="0.5405"/>
-	<xacro:property name="def_torso_roll" value="0"/>
-	<xacro:property name="def_torso_pitch" value="0"/>
-	<xacro:property name="def_torso_yaw" value="-0.445"/>
+	<xacro:property name="def_torso_roll" value="0.0"/>
+	<xacro:property name="def_torso_pitch" value="0.0"/>
+	<xacro:property name="def_torso_yaw" value="0.0"/>
 	<!-- head mount positions | relative to head_cover_link -->
 	<xacro:property name="def_head_x" value="0.0"/>

File: cob_hardware_config/robots/raw3-1/urdf/raw3-1.urdf.xacro (robot description, xacro)
@@ -11,11 +11,9 @@
   <xacro:include filename="$(find raw_description)/urdf/tower_asymetric/tower.urdf.xacro" />
   <!-- torso -->
-  <xacro:include filename="$(find raw_description)/urdf/torso/torso.urdf.xacro" />
-  <!-- head -->
-  <xacro:include filename="$(find raw_description)/urdf/head/head.urdf.xacro" />
+  <xacro:include filename="$(find raw_description)/urdf/torso/torso_v2.urdf.xacro" />
   <!-- ur_arm -->
-  <xacro:include filename="$(find raw_description)/urdf/ur_arm/ur10_arm.urdf.xacro" />
+  <!--xacro:include filename="$(find raw_description)/urdf/ur_arm/ur10_arm.urdf.xacro" /-->
   <!-- vacuum gripper -->
-  <xacro:include filename="$(find raw_description)/urdf/vacuum_gripper/gripper.urdf.xacro" />
+  <!--xacro:include filename="$(find raw_description)/urdf/vacuum_gripper/gripper.urdf.xacro" /-->
   <!-- sensors -->
   <xacro:include filename="$(find cob_description)/urdf/sensors/sick_s300_laser.urdf.xacro"/>
@@ -33,15 +31,12 @@
     <origin xyz="${tower_x} ${tower_y} ${tower_z}" rpy="${tower_roll} ${tower_pitch} ${tower_yaw}" />
   </xacro:tower_asymetric>
-  <xacro:raw_torso name="torso" parent="base_link">
+  <xacro:raw_torso_v2 name="torso" parent="base_link">
     <origin xyz="${torso_x} ${torso_y} ${torso_z}" rpy="${torso_roll} ${torso_pitch} ${torso_yaw}" />
-  </xacro:raw_torso>
-  <xacro:raw_head name="head" parent="torso_2_link">
-    <origin xyz="${head_x} ${head_y} ${head_z}" rpy="${head_roll} ${head_pitch} ${head_yaw}" />
-  </xacro:raw_head>
-  <xacro:ur10 name="arm" parent="base_link">
+  </xacro:raw_torso_v2>
+  <!--xacro:ur10 name="arm" parent="base_link">
     <origin xyz="${arm_x} ${arm_y} ${arm_z}" rpy="${arm_roll} ${arm_pitch} ${arm_yaw}" />
-  </xacro:ur10>
-  <xacro:vacuum_gripper name="gripper" parent="arm_ee_link">
+  </xacro:ur10-->
+  <!--xacro:vacuum_gripper name="gripper" parent="arm_ee_link">
     <origin xyz="${gripper_x} ${gripper_y} ${gripper_z}" rpy="${gripper_roll} ${gripper_pitch} ${gripper_yaw}" />
-  </xacro:vacuum_gripper>
+  </xacro:vacuum_gripper-->
 </robot>

Commit message: merge new stuff with working branch on robot

File: cob_hardware_config/robots/raw3-1/urdf/calibration_default.urdf.xacro (robot description, xacro)
@@ -87,3 +87,10 @@
 	<xacro:property name="def_cam3d_pitch" value="0.0"/>
 	<xacro:property name="def_cam3d_yaw" value="0.0"/>
+        <!-- arm camera | handeye calibration | relative to cam_reference_link -->
+        <xacro:property name="def_arm_camera_x" value="0.00"/>
+        <xacro:property name="def_arm_camera_y" value="0.0"/>
+        <xacro:property name="def_arm_camera_z" value="0.0"/>
+        <xacro:property name="def_arm_camera_roll" value="0.0"/>
+        <xacro:property name="def_arm_camera_pitch" value="0.0"/>
+        <xacro:property name="def_arm_camera_yaw" value="0.0"/>
 </robot>

File: cob_hardware_config/robots/raw3-1/urdf/properties.urdf.xacro (robot description, xacro)
@@ -89,3 +89,10 @@
 	<xacro:property name="cam3d_pitch" value="${def_cam3d_pitch+offset_cam3d_pitch}"/>
 	<xacro:property name="cam3d_yaw" value="${def_cam3d_yaw+offset_cam3d_yaw}"/>
+        <!-- arm camera | handeye calibration | relative to cam_reference_link -->
+        <xacro:property name="arm_camera_x" value="${def_arm_camera_x}"/>
+        <xacro:property name="arm_camera_y" value="${def_arm_camera_y}"/>
+        <xacro:property name="arm_camera_z" value="${def_arm_camera_z}"/>
+        <xacro:property name="arm_camera_roll" value="${def_arm_camera_roll}"/>
+        <xacro:property name="arm_camera_pitch" value="${def_arm_camera_pitch}"/>
+        <xacro:property name="arm_camera_yaw" value="${def_arm_camera_yaw}"/>
 </robot>

File: cob_hardware_config/robots/raw3-1/urdf/raw3-1.urdf.xacro (robot description, xacro)
@@ -15,5 +15,9 @@
   <xacro:include filename="$(find raw_description)/urdf/ur_arm/ur10_arm.urdf.xacro" />
   <!-- vacuum gripper -->
-  <xacro:include filename="$(find raw_description)/urdf/vacuum_gripper/gripper.urdf.xacro" />
+  <!--xacro:include filename="$(find raw_description)/urdf/vacuum_gripper/gripper.urdf.xacro" /-->
+  <!-- schmaltz vacuum gripper -->
+  <xacro:include filename="$(find raw_description)/urdf/schmaltz_gripper/gripper.urdf.xacro" />
+  <!-- arm camera -->
+  <xacro:include filename="$(find raw_description)/urdf/arm_camera/arm_camera.urdf.xacro" />
   <!-- sensors -->
   <xacro:include filename="$(find cob_description)/urdf/sensors/sick_s300_laser.urdf.xacro"/>
