Commit message: replace ur_arm with p_rob_arm

File: cob_hardware_config/robots/raw3-1/urdf/raw3-1.urdf.xacro (robot description, xacro)
@@ -14,8 +14,6 @@
   <!-- head -->
   <xacro:include filename="$(find raw_description)/urdf/head/head.urdf.xacro" />
-  <!-- ur_arm -->
-  <xacro:include filename="$(find cob_description)/urdf/ur_arm/ur10_arm.urdf.xacro" />
-  <!-- vacuum gripper -->
-  <xacro:include filename="$(find raw_description)/urdf/vacuum_gripper/gripper.urdf.xacro" />
+  <!-- p_rob -->
+  <xacro:include filename="$(find cob_description)/urdf/p_rob/p_rob.urdf.xacro" />
   <!-- sensors -->
   <xacro:include filename="$(find cob_description)/urdf/sensors/sick_s300_laser.urdf.xacro"/>
@@ -39,9 +37,6 @@
     <origin xyz="${head_x} ${head_y} ${head_z}" rpy="${head_roll} ${head_pitch} ${head_yaw}" />
   </xacro:raw_head>
-  <xacro:ur10 name="arm" parent="base_link">
+  <xacro:p_rob name="arm" parent="base_link">
     <origin xyz="${arm_x} ${arm_y} ${arm_z}" rpy="${arm_roll} ${arm_pitch} ${arm_yaw}" />
-  </xacro:ur10>
-  <xacro:vacuum_gripper name="gripper" parent="arm_ee_link">
-    <origin xyz="${gripper_x} ${gripper_y} ${gripper_z}" rpy="${gripper_roll} ${gripper_pitch} ${gripper_yaw}" />
-  </xacro:vacuum_gripper>
+  </xacro:p_rob>
 </robot>

Commit message: undo changes for p_rob joint name

File: cob_hardware_config/robots/raw3-1/urdf/raw3-1.urdf.xacro (robot description, xacro)
@@ -14,6 +14,8 @@
   <!-- head -->
   <xacro:include filename="$(find raw_description)/urdf/head/head.urdf.xacro" />
-  <!-- p_rob -->
-  <xacro:include filename="$(find cob_description)/urdf/p_rob/p_rob.urdf.xacro" />
+  <!-- ur_arm -->
+  <xacro:include filename="$(find cob_description)/urdf/ur_arm/ur10_arm.urdf.xacro" />
+  <!-- vacuum gripper -->
+  <xacro:include filename="$(find raw_description)/urdf/vacuum_gripper/gripper.urdf.xacro" />
   <!-- sensors -->
   <xacro:include filename="$(find cob_description)/urdf/sensors/sick_s300_laser.urdf.xacro"/>
@@ -37,6 +39,9 @@
     <origin xyz="${head_x} ${head_y} ${head_z}" rpy="${head_roll} ${head_pitch} ${head_yaw}" />
   </xacro:raw_head>
-  <xacro:p_rob name="arm" parent="base_link">
+  <xacro:ur10 name="arm" parent="base_link">
     <origin xyz="${arm_x} ${arm_y} ${arm_z}" rpy="${arm_roll} ${arm_pitch} ${arm_yaw}" />
-  </xacro:p_rob>
+  </xacro:ur10>
+  <xacro:vacuum_gripper name="gripper" parent="arm_ee_link">
+    <origin xyz="${gripper_x} ${gripper_y} ${gripper_z}" rpy="${gripper_roll} ${gripper_pitch} ${gripper_yaw}" />
+  </xacro:vacuum_gripper>
 </robot>

Commit message: update kinetic camera

File: cob_hardware_config/robots/raw3-1/urdf/raw3-1.urdf.xacro (robot description, xacro)
@@ -44,3 +44,6 @@
     <origin xyz="${gripper_x} ${gripper_y} ${gripper_z}" rpy="${gripper_roll} ${gripper_pitch} ${gripper_yaw}" />
   </xacro:vacuum_gripper>
+  <xacro:kinect_camera name="arm_camera" ros_topic="arm_kinect_camera" parent="gripper_coupling_link" update_rate="30" data_skip="9">
+    <origin xyz="${arm_camera_x} ${arm_camera_y} ${arm_camera_z}" rpy="${arm_camera_roll} ${arm_camera_pitch} ${arm_camera_yaw}" />
+  </xacro:kinect_camera>
 </robot>
