Commit message: make same file and offset value as other camera

File: cob_hardware_config/robots/cob4-7/urdf/properties.urdf.xacro (robot description, xacro)
@@ -106,9 +106,9 @@
 	<xacro:property name="head_cam_yaw" value="${def_head_cam_yaw+offset_head_cam_yaw}"/>
         <!-- cam | handeye calibration | relative to head_3_link -->
-        <xacro:property name="face_cam_x" value="${def_face_cam_x}"/>
-        <xacro:property name="face_cam_y" value="${def_face_cam_y}"/>
-        <xacro:property name="face_cam_z" value="${def_face_cam_z}"/>
-        <xacro:property name="face_cam_roll" value="${def_face_cam_roll}"/>
-        <xacro:property name="face_cam_pitch" value="${def_face_cam_pitch}"/>
-        <xacro:property name="face_cam_yaw" value="${def_face_cam_yaw}"/>
+        <xacro:property name="face_cam_x" value="${def_face_cam_x+offset_face_cam_x}"/>
+        <xacro:property name="face_cam_y" value="${def_face_cam_y+offset_face_cam_y}"/>
+        <xacro:property name="face_cam_z" value="${def_face_cam_z+offset_face_cam_z}"/>
+        <xacro:property name="face_cam_roll" value="${def_face_cam_roll+offset_face_cam_roll}"/>
+        <xacro:property name="face_cam_pitch" value="${def_face_cam_pitch+offset_face_cam_pitch}"/>
+        <xacro:property name="face_cam_yaw" value="${def_face_cam_yaw+offset_face_cam_yaw}"/>
 </robot>

Commit message: add face cam

File: cob_hardware_config/robots/cob4-7/urdf/properties.urdf.xacro (robot description, xacro)
@@ -119,3 +119,10 @@
 	<xacro:property name="head_cam_pitch" value="${def_head_cam_pitch+offset_head_cam_pitch}"/>
 	<xacro:property name="head_cam_yaw" value="${def_head_cam_yaw+offset_head_cam_yaw}"/>
+        <!-- cam | handeye calibration | relative to head_3_link -->
+        <xacro:property name="face_cam_x" value="${def_face_cam_x+offset_face_cam_x}"/>
+        <xacro:property name="face_cam_y" value="${def_face_cam_y+offset_face_cam_y}"/>
+        <xacro:property name="face_cam_z" value="${def_face_cam_z+offset_face_cam_z}"/>
+        <xacro:property name="face_cam_roll" value="${def_face_cam_roll+offset_face_cam_roll}"/>
+        <xacro:property name="face_cam_pitch" value="${def_face_cam_pitch+offset_face_cam_pitch}"/>
+        <xacro:property name="face_cam_yaw" value="${def_face_cam_yaw+offset_face_cam_yaw}"/>
 </robot>
