Commit message: add face camera calibration and urdf

File: cob_hardware_config/robots/cob4-7/urdf/calibration_default.urdf.xacro (robot description, xacro)
@@ -102,3 +102,10 @@
 	<xacro:property name="def_head_cam_pitch" value="-0.73"/>
 	<xacro:property name="def_head_cam_yaw" value="0.0"/>
+        <!-- cam | handeye calibration | relative to head_3_link -->
+        <xacro:property name="def_face_cam_x" value="-0.18486"/>
+        <xacro:property name="def_face_cam_y" value="0.0"/>
+        <xacro:property name="def_face_cam_z" value="0.38953"/>
+        <xacro:property name="def_face_cam_roll" value="0.0"/> <!-- -1.57079 -->
+        <xacro:property name="def_face_cam_pitch" value="-0.1745"/>
+        <xacro:property name="def_face_cam_yaw" value="0.0"/>
 </robot>

File: cob_hardware_config/robots/cob4-7/urdf/cob4-7.urdf.xacro (robot description, xacro)
@@ -58,4 +58,7 @@
     <origin xyz="${head_cam_x} ${head_cam_y} ${head_cam_z}" rpy="${head_cam_roll} ${head_cam_pitch} ${head_cam_yaw}" />
   </xacro:usb_cam>
+  <xacro:realsense name="face_cam" ros_topic="face_cam" parent="head_3_link">
+    <origin xyz="${face_cam_x} ${face_cam_y} ${face_cam_z}" rpy="${face_cam_roll} ${face_cam_pitch} ${face_cam_yaw}" />
+  </xacro:realsense>
   <!--xacro:cob4_arm name="arm_right" parent="torso_3_link" has_podest="false">
     <origin xyz="${arm_right_x} ${arm_right_y} ${arm_right_z}" rpy="${arm_right_roll} ${arm_right_pitch} ${arm_right_yaw}" />

File: cob_hardware_config/robots/cob4-7/urdf/properties.urdf.xacro (robot description, xacro)
@@ -105,3 +105,10 @@
 	<xacro:property name="head_cam_pitch" value="${def_head_cam_pitch+offset_head_cam_pitch}"/>
 	<xacro:property name="head_cam_yaw" value="${def_head_cam_yaw+offset_head_cam_yaw}"/>
+        <!-- cam | handeye calibration | relative to head_3_link -->
+        <xacro:property name="face_cam_x" value="${def_face_cam_x}"/>
+        <xacro:property name="face_cam_y" value="${def_face_cam_y}"/>
+        <xacro:property name="face_cam_z" value="${def_face_cam_z}"/>
+        <xacro:property name="face_cam_roll" value="${def_face_cam_roll}"/>
+        <xacro:property name="face_cam_pitch" value="${def_face_cam_pitch}"/>
+        <xacro:property name="face_cam_yaw" value="${def_face_cam_yaw}"/>
 </robot>

Commit message: gripper calibration and add door open position

File: cob_hardware_config/robots/cob4-7/urdf/calibration_default.urdf.xacro (robot description, xacro)
@@ -63,4 +63,18 @@
 	<xacro:property name="def_arm_left_pitch" value="0"/>
 	<xacro:property name="def_arm_left_yaw" value="3.14159"/>
+        <!-- gripper right mount positions | relative to arm_right_7_link -->
+        <xacro:property name="def_gripper_right_x" value="0.0"/>
+        <xacro:property name="def_gripper_right_y" value="0.0"/>
+        <xacro:property name="def_gripper_right_z" value="0.0748"/>
+        <xacro:property name="def_gripper_right_roll" value="0.0"/>
+        <xacro:property name="def_gripper_right_pitch" value="0.0"/>
+        <xacro:property name="def_gripper_right_yaw" value="3.14159"/>
+        <!-- gripper left mount positions | relative to arm_left_7_link -->
+        <xacro:property name="def_gripper_left_x" value="0.0"/>
+        <xacro:property name="def_gripper_left_y" value="0.0"/>
+        <xacro:property name="def_gripper_left_z" value="0.0748"/>
+        <xacro:property name="def_gripper_left_roll" value="0.0"/>
+        <xacro:property name="def_gripper_left_pitch" value="0.0"/>
+        <xacro:property name="def_gripper_left_yaw" value="3.14159"/>
 	<!-- *********************************** -->
 	<!-- kinematic chain reference positions -->

File: cob_hardware_config/robots/cob4-7/urdf/cob4-7.urdf.xacro (robot description, xacro)
@@ -61,7 +61,7 @@
     <origin xyz="${arm_right_x} ${arm_right_y} ${arm_right_z}" rpy="${arm_right_roll} ${arm_right_pitch} ${arm_right_yaw}" />
   </xacro:cob4_arm>
-  <xacro:cob4_arm name="arm_left" parent="torso_3_link" has_podest="false">
+  <!--xacro:cob4_arm name="arm_left" parent="torso_3_link" has_podest="false">
     <origin xyz="${arm_left_x} ${arm_left_y} ${arm_left_z}" rpy="${arm_left_roll} ${arm_left_pitch} ${arm_left_yaw}" />
-  </xacro:cob4_arm>
+  </xacro:cob4_arm-->
   <xacro:sensorring name="sensorring" parent="head_3_link" active="false">  <!-- HotFix: set active to true when the HW is repaired -->
     <origin xyz="${sensorring_x} ${sensorring_y} ${sensorring_z}" rpy="${sensorring_roll} ${sensorring_pitch} ${sensorring_yaw}" />
@@ -70,3 +70,6 @@
     <origin xyz="${sensorring_cam3d_x} ${sensorring_cam3d_y} ${sensorring_cam3d_z}" rpy="${sensorring_cam3d_roll} ${sensorring_cam3d_pitch} ${sensorring_cam3d_yaw}" />
   </xacro:cob_kinect_v0>
+  <xacro:gripper name="gripper_right" parent="arm_right_7_link">
+    <origin xyz="${gripper_right_x} ${gripper_right_y} ${gripper_right_z}" rpy="${gripper_right_roll} ${gripper_right_pitch} ${gripper_right_yaw}" />
+  </xacro:gripper>
 </robot>

File: cob_hardware_config/robots/cob4-7/urdf/properties.urdf.xacro (robot description, xacro)
@@ -66,4 +66,18 @@
 	<xacro:property name="arm_left_pitch" value="${def_arm_left_pitch+offset_arm_left_pitch}"/>
 	<xacro:property name="arm_left_yaw" value="${def_arm_left_yaw+offset_arm_left_yaw}"/>
+        <!-- gripper mount positions | relative to arm_7_link -->
+        <xacro:property name="gripper_right_x" value="${def_gripper_right_x+offset_gripper_right_x}"/>
+        <xacro:property name="gripper_right_y" value="${def_gripper_right_y+offset_gripper_right_y}"/>
+        <xacro:property name="gripper_right_z" value="${def_gripper_right_z+offset_gripper_right_z}"/>
+        <xacro:property name="gripper_right_roll" value="${def_gripper_right_roll+offset_gripper_right_roll}"/>
+        <xacro:property name="gripper_right_pitch" value="${def_gripper_right_pitch+offset_gripper_right_pitch}"/>
+        <xacro:property name="gripper_right_yaw" value="${def_gripper_right_yaw+offset_gripper_right_yaw}"/>
+        <!-- gripper mount positions | relative to arm_7_link -->
+        <xacro:property name="gripper_left_x" value="${def_gripper_left_x+offset_gripper_left_x}"/>
+        <xacro:property name="gripper_left_y" value="${def_gripper_left_y+offset_gripper_left_y}"/>
+        <xacro:property name="gripper_left_z" value="${def_gripper_left_z+offset_gripper_left_z}"/>
+        <xacro:property name="gripper_left_roll" value="${def_gripper_left_roll+offset_gripper_left_roll}"/>
+        <xacro:property name="gripper_left_pitch" value="${def_gripper_left_pitch+offset_gripper_left_pitch}"/>
+        <xacro:property name="gripper_left_yaw" value="${def_gripper_left_yaw+offset_gripper_left_yaw}"/>
 	<!-- *********************************** -->
 	<!-- kinematic chain reference positions -->

Commit message: added hand_mounting in calibration

File: cob_hardware_config/robots/cob4-7/urdf/calibration_default.urdf.xacro (robot description, xacro)
@@ -63,4 +63,18 @@
 	<xacro:property name="def_arm_left_pitch" value="0"/>
 	<xacro:property name="def_arm_left_yaw" value="3.14159"/>
+	<!-- gripper right mount positions | relative to arm_right_7_link -->
+	<xacro:property name="def_gripper_right_x" value="0.0"/>
+	<xacro:property name="def_gripper_right_y" value="0.0"/>
+	<xacro:property name="def_gripper_right_z" value="0.0748"/>
+	<xacro:property name="def_gripper_right_roll" value="0.0"/>
+	<xacro:property name="def_gripper_right_pitch" value="0.0"/>
+	<xacro:property name="def_gripper_right_yaw" value="3.14159"/>
+	<!-- gripper left mount positions | relative to arm_left_7_link -->
+	<xacro:property name="def_gripper_left_x" value="0.0"/>
+	<xacro:property name="def_gripper_left_y" value="0.0"/>
+	<xacro:property name="def_gripper_left_z" value="0.0748"/>
+	<xacro:property name="def_gripper_left_roll" value="0.0"/>
+	<xacro:property name="def_gripper_left_pitch" value="0.0"/>
+	<xacro:property name="def_gripper_left_yaw" value="3.14159"/>
 	<!-- ***************************** -->
 	<!-- extrinsic camera calibration  -->

Commit message: add gripper urdf

File: cob_hardware_config/robots/cob4-7/urdf/calibration_default.urdf.xacro (robot description, xacro)
@@ -63,5 +63,19 @@
 	<xacro:property name="def_arm_left_pitch" value="0"/>
 	<xacro:property name="def_arm_left_yaw" value="3.14159"/>
-	<!-- ***************************** -->
+        <!-- gripper right mount positions | relative to arm_right_7_link -->
+        <xacro:property name="def_gripper_right_x" value="0.0"/>
+        <xacro:property name="def_gripper_right_y" value="0.0"/>
+        <xacro:property name="def_gripper_right_z" value="0.0748"/>
+        <xacro:property name="def_gripper_right_roll" value="0.0"/>
+        <xacro:property name="def_gripper_right_pitch" value="0.0"/>
+        <xacro:property name="def_gripper_right_yaw" value="3.14159"/>
+        <!-- gripper left mount positions | relative to arm_left_7_link -->
+        <xacro:property name="def_gripper_left_x" value="0.0"/>
+        <xacro:property name="def_gripper_left_y" value="0.0"/>
+        <xacro:property name="def_gripper_left_z" value="0.0748"/>
+        <xacro:property name="def_gripper_left_roll" value="0.0"/>
+        <xacro:property name="def_gripper_left_pitch" value="0.0"/>
+        <xacro:property name="def_gripper_left_yaw" value="3.14159"/>
+        <!-- ***************************** -->
 	<!-- extrinsic camera calibration  -->
 	<!-- ***************************** -->

File: cob_hardware_config/robots/cob4-7/urdf/cob4-7.urdf.xacro (robot description, xacro)
@@ -67,4 +67,10 @@
     <origin xyz="${arm_left_x} ${arm_left_y} ${arm_left_z}" rpy="${arm_left_roll} ${arm_left_pitch} ${arm_left_yaw}" />
   </xacro:cob4_arm>
+  <xacro:gripper name="gripper_right" parent="arm_right_7_link">
+    <origin xyz="${gripper_right_x} ${gripper_right_y} ${gripper_right_z}" rpy="${gripper_right_roll} ${gripper_right_pitch} ${gripper_right_yaw}" />
+  </xacro:gripper>
+  <xacro:gripper name="gripper_left" parent="arm_left_7_link">
+    <origin xyz="${gripper_left_x} ${gripper_left_y} ${gripper_left_z}" rpy="${gripper_left_roll} ${gripper_left_pitch} ${gripper_left_yaw}" />
+  </xacro:gripper>
   <xacro:sensorring name="sensorring" parent="head_3_link" active="true">
     <origin xyz="${sensorring_x} ${sensorring_y} ${sensorring_z}" rpy="${sensorring_roll} ${sensorring_pitch} ${sensorring_yaw}" />

File: cob_hardware_config/robots/cob4-7/urdf/properties.urdf.xacro (robot description, xacro)
@@ -66,5 +66,19 @@
 	<xacro:property name="arm_left_pitch" value="${def_arm_left_pitch+offset_arm_left_pitch}"/>
 	<xacro:property name="arm_left_yaw" value="${def_arm_left_yaw+offset_arm_left_yaw}"/>
-	<!-- *********************************** -->
+        <!-- gripper mount positions | relative to arm_7_link -->
+        <xacro:property name="gripper_right_x" value="${def_gripper_right_x+offset_gripper_right_x}"/>
+        <xacro:property name="gripper_right_y" value="${def_gripper_right_y+offset_gripper_right_y}"/>
+        <xacro:property name="gripper_right_z" value="${def_gripper_right_z+offset_gripper_right_z}"/>
+        <xacro:property name="gripper_right_roll" value="${def_gripper_right_roll+offset_gripper_right_roll}"/>
+        <xacro:property name="gripper_right_pitch" value="${def_gripper_right_pitch+offset_gripper_right_pitch}"/>
+        <xacro:property name="gripper_right_yaw" value="${def_gripper_right_yaw+offset_gripper_right_yaw}"/>
+        <!-- gripper mount positions | relative to arm_7_link -->
+        <xacro:property name="gripper_left_x" value="${def_gripper_left_x+offset_gripper_left_x}"/>
+        <xacro:property name="gripper_left_y" value="${def_gripper_left_y+offset_gripper_left_y}"/>
+        <xacro:property name="gripper_left_z" value="${def_gripper_left_z+offset_gripper_left_z}"/>
+        <xacro:property name="gripper_left_roll" value="${def_gripper_left_roll+offset_gripper_left_roll}"/>
+        <xacro:property name="gripper_left_pitch" value="${def_gripper_left_pitch+offset_gripper_left_pitch}"/>
+        <xacro:property name="gripper_left_yaw" value="${def_gripper_left_yaw+offset_gripper_left_yaw}"/>
+        <!-- *********************************** -->
 	<!-- kinematic chain reference positions -->
 	<!-- *********************************** -->
