Commit message: fast test not know which is correct

File: cob_hardware_config/robots/cob4-7/urdf/calibration_default.urdf.xacro (robot description, xacro)
@@ -63,37 +63,50 @@
 	<xacro:property name="def_arm_left_pitch" value="0"/>
 	<xacro:property name="def_arm_left_yaw" value="3.14159"/>
-	<!-- *********************************** -->
-	<!-- kinematic chain reference positions -->
-	<!-- *********************************** -->
-	<!-- this feature is no longer supported as urdfdom does not parse the according 'calibration_rising' tag -->
-	<!-- cam3d left | handeye calibration | relative to torso_3_link -->
-	<xacro:property name="def_torso_cam3d_left_x" value="0.12839"/>
-	<xacro:property name="def_torso_cam3d_left_y" value="0.01802"/>
-	<xacro:property name="def_torso_cam3d_left_z" value="0.24214"/>
-	<xacro:property name="def_torso_cam3d_left_roll" value="1.57079"/>
+        <!-- gripper right mount positions | relative to arm_right_7_link -->
+        <xacro:property name="def_gripper_right_x" value="0.0"/>
+        <xacro:property name="def_gripper_right_y" value="0.0"/>
+        <xacro:property name="def_gripper_right_z" value="0.0748"/>
+        <xacro:property name="def_gripper_right_roll" value="0.0"/>
+        <xacro:property name="def_gripper_right_pitch" value="0.0"/>
+        <xacro:property name="def_gripper_right_yaw" value="3.14159"/>
+        <!-- gripper left mount positions | relative to arm_left_7_link -->
+        <xacro:property name="def_gripper_left_x" value="0.0"/>
+        <xacro:property name="def_gripper_left_y" value="0.0"/>
+        <xacro:property name="def_gripper_left_z" value="0.0748"/>
+        <xacro:property name="def_gripper_left_roll" value="0.0"/>
+        <xacro:property name="def_gripper_left_pitch" value="0.0"/>
+        <xacro:property name="def_gripper_left_yaw" value="3.14159"/>
+        <!-- ***************************** -->
+	<!-- extrinsic camera calibration  -->
+	<!-- ***************************** -->
+	<!-- torso cam3d left mount positions | relative to torso_3_link -->
+	<xacro:property name="def_torso_cam3d_left_x" value="0.14873"/>
+	<xacro:property name="def_torso_cam3d_left_y" value="0.01293"/>
+	<xacro:property name="def_torso_cam3d_left_z" value="0.27008"/>
+	<xacro:property name="def_torso_cam3d_left_roll" value="-1.57079"/>
 	<xacro:property name="def_torso_cam3d_left_pitch" value="0.0"/>
-	<xacro:property name="def_torso_cam3d_left_yaw" value="0.418879"/>
-	<!-- cam3d right | handeye calibration | relative to torso_3_link -->
-	<xacro:property name="def_torso_cam3d_right_x" value="0.12839"/>
-	<xacro:property name="def_torso_cam3d_right_y" value="-0.01802"/>
-	<xacro:property name="def_torso_cam3d_right_z" value="0.24214"/>
-	<xacro:property name="def_torso_cam3d_right_roll" value="1.57079"/>
+	<xacro:property name="def_torso_cam3d_left_yaw" value="0.61"/>
+	<!-- torso cam3d right mount positions | relative to torso_3_link -->
+	<xacro:property name="def_torso_cam3d_right_x" value="0.14873"/>
+	<xacro:property name="def_torso_cam3d_right_y" value="-0.01293"/>
+	<xacro:property name="def_torso_cam3d_right_z" value="0.27008"/>
+	<xacro:property name="def_torso_cam3d_right_roll" value="-1.57079"/>
 	<xacro:property name="def_torso_cam3d_right_pitch" value="0.0"/>
-	<xacro:property name="def_torso_cam3d_right_yaw" value="-0.418879"/>
-	<!-- cam3d down | handeye calibration | relative to torso_3_link -->
-	<xacro:property name="def_torso_cam3d_down_x" value="0.15908"/>
+	<xacro:property name="def_torso_cam3d_right_yaw" value="-0.61"/>
+	<!-- torso cam3d down mount positions | relative to torso_3_link -->
+	<xacro:property name="def_torso_cam3d_down_x" value="0.15203"/>
 	<xacro:property name="def_torso_cam3d_down_y" value="0.0"/>
-	<xacro:property name="def_torso_cam3d_down_z" value="0.14005"/>
+	<xacro:property name="def_torso_cam3d_down_z" value="0.1307"/>
 	<xacro:property name="def_torso_cam3d_down_roll" value="0.0"/>
-	<xacro:property name="def_torso_cam3d_down_pitch" value="0.61086"/>
+	<xacro:property name="def_torso_cam3d_down_pitch" value="0.56"/>
 	<xacro:property name="def_torso_cam3d_down_yaw" value="0.0"/>
-	<!-- cam3d | handeye calibration | relative to sensorring_link -->
-	<xacro:property name="def_sensorring_cam3d_x" value="0.096"/>
+	<!-- sensorring cam3d mount positions | relative to sensorring_link -->
+	<xacro:property name="def_sensorring_cam3d_x" value="0.1251"/>
 	<xacro:property name="def_sensorring_cam3d_y" value="0.0"/>
-	<xacro:property name="def_sensorring_cam3d_z" value="0.0195"/>
+	<xacro:property name="def_sensorring_cam3d_z" value="0.001"/>
 	<xacro:property name="def_sensorring_cam3d_roll" value="0.0"/>
 	<xacro:property name="def_sensorring_cam3d_pitch" value="0.0"/>
 	<xacro:property name="def_sensorring_cam3d_yaw" value="0.0"/>
-	<!-- cam | handeye calibration | relative to head_3_link -->
+	<!-- head cam mount positions | relative to head_3_link -->
 	<xacro:property name="def_head_cam_x" value="-0.181"/>
 	<xacro:property name="def_head_cam_y" value="0.0"/>
@@ -102,3 +115,10 @@
 	<xacro:property name="def_head_cam_pitch" value="-0.73"/>
 	<xacro:property name="def_head_cam_yaw" value="0.0"/>
+        <!-- cam | handeye calibration | relative to head_3_link -->
+        <xacro:property name="def_face_cam_x" value="-0.18486"/>
+        <xacro:property name="def_face_cam_y" value="0.0"/>
+        <xacro:property name="def_face_cam_z" value="0.38953"/>
+        <xacro:property name="def_face_cam_roll" value="0.0"/> <!-- -1.57079 -->
+        <xacro:property name="def_face_cam_pitch" value="-0.1745"/>
+        <xacro:property name="def_face_cam_yaw" value="0.0"/>
 </robot>

File: cob_hardware_config/robots/cob4-7/urdf/cob4-7.urdf.xacro (robot description, xacro)
@@ -58,11 +58,20 @@
     <origin xyz="${head_cam_x} ${head_cam_y} ${head_cam_z}" rpy="${head_cam_roll} ${head_cam_pitch} ${head_cam_yaw}" />
   </xacro:usb_cam>
-  <!--xacro:cob4_arm name="arm_right" parent="torso_3_link" has_podest="false">
+  <xacro:realsense name="face_cam" ros_topic="face_cam" parent="head_3_link">
+    <origin xyz="${face_cam_x} ${face_cam_y} ${face_cam_z}" rpy="${face_cam_roll} ${face_cam_pitch} ${face_cam_yaw}" />
+  </xacro:realsense>
+  <xacro:cob4_arm name="arm_right" parent="torso_3_link" has_podest="false">
     <origin xyz="${arm_right_x} ${arm_right_y} ${arm_right_z}" rpy="${arm_right_roll} ${arm_right_pitch} ${arm_right_yaw}" />
   </xacro:cob4_arm>
   <xacro:cob4_arm name="arm_left" parent="torso_3_link" has_podest="false">
     <origin xyz="${arm_left_x} ${arm_left_y} ${arm_left_z}" rpy="${arm_left_roll} ${arm_left_pitch} ${arm_left_yaw}" />
-  </xacro:cob4_arm-->
-  <xacro:sensorring name="sensorring" parent="head_3_link" active="false">  <!-- HotFix: set active to true when the HW is repaired -->
+  </xacro:cob4_arm>
+  <xacro:gripper name="gripper_right" parent="arm_right_7_link">
+    <origin xyz="${gripper_right_x} ${gripper_right_y} ${gripper_right_z}" rpy="${gripper_right_roll} ${gripper_right_pitch} ${gripper_right_yaw}" />
+  </xacro:gripper>
+  <xacro:gripper name="gripper_left" parent="arm_left_7_link">
+    <origin xyz="${gripper_left_x} ${gripper_left_y} ${gripper_left_z}" rpy="${gripper_left_roll} ${gripper_left_pitch} ${gripper_left_yaw}" />
+  </xacro:gripper>
+  <xacro:sensorring name="sensorring" parent="head_3_link" active="true">
     <origin xyz="${sensorring_x} ${sensorring_y} ${sensorring_z}" rpy="${sensorring_roll} ${sensorring_pitch} ${sensorring_yaw}" />
   </xacro:sensorring>

File: cob_hardware_config/robots/cob4-7/urdf/properties.urdf.xacro (robot description, xacro)
@@ -66,5 +66,19 @@
 	<xacro:property name="arm_left_pitch" value="${def_arm_left_pitch+offset_arm_left_pitch}"/>
 	<xacro:property name="arm_left_yaw" value="${def_arm_left_yaw+offset_arm_left_yaw}"/>
-	<!-- *********************************** -->
+        <!-- gripper mount positions | relative to arm_7_link -->
+        <xacro:property name="gripper_right_x" value="${def_gripper_right_x+offset_gripper_right_x}"/>
+        <xacro:property name="gripper_right_y" value="${def_gripper_right_y+offset_gripper_right_y}"/>
+        <xacro:property name="gripper_right_z" value="${def_gripper_right_z+offset_gripper_right_z}"/>
+        <xacro:property name="gripper_right_roll" value="${def_gripper_right_roll+offset_gripper_right_roll}"/>
+        <xacro:property name="gripper_right_pitch" value="${def_gripper_right_pitch+offset_gripper_right_pitch}"/>
+        <xacro:property name="gripper_right_yaw" value="${def_gripper_right_yaw+offset_gripper_right_yaw}"/>
+        <!-- gripper mount positions | relative to arm_7_link -->
+        <xacro:property name="gripper_left_x" value="${def_gripper_left_x+offset_gripper_left_x}"/>
+        <xacro:property name="gripper_left_y" value="${def_gripper_left_y+offset_gripper_left_y}"/>
+        <xacro:property name="gripper_left_z" value="${def_gripper_left_z+offset_gripper_left_z}"/>
+        <xacro:property name="gripper_left_roll" value="${def_gripper_left_roll+offset_gripper_left_roll}"/>
+        <xacro:property name="gripper_left_pitch" value="${def_gripper_left_pitch+offset_gripper_left_pitch}"/>
+        <xacro:property name="gripper_left_yaw" value="${def_gripper_left_yaw+offset_gripper_left_yaw}"/>
+        <!-- *********************************** -->
 	<!-- kinematic chain reference positions -->
 	<!-- *********************************** -->
@@ -105,3 +119,10 @@
 	<xacro:property name="head_cam_pitch" value="${def_head_cam_pitch+offset_head_cam_pitch}"/>
 	<xacro:property name="head_cam_yaw" value="${def_head_cam_yaw+offset_head_cam_yaw}"/>
+        <!-- cam | handeye calibration | relative to head_3_link -->
+        <xacro:property name="face_cam_x" value="${def_face_cam_x+offset_face_cam_x}"/>
+        <xacro:property name="face_cam_y" value="${def_face_cam_y+offset_face_cam_y}"/>
+        <xacro:property name="face_cam_z" value="${def_face_cam_z+offset_face_cam_z}"/>
+        <xacro:property name="face_cam_roll" value="${def_face_cam_roll+offset_face_cam_roll}"/>
+        <xacro:property name="face_cam_pitch" value="${def_face_cam_pitch+offset_face_cam_pitch}"/>
+        <xacro:property name="face_cam_yaw" value="${def_face_cam_yaw+offset_face_cam_yaw}"/>
 </robot>

File: cob_hardware_config/robots/raw3-1/urdf/raw3-1.urdf.xacro (robot description, xacro)
@@ -15,5 +15,9 @@
   <xacro:include filename="$(find raw_description)/urdf/ur_arm/ur10_arm.urdf.xacro" />
   <!-- vacuum gripper -->
-  <xacro:include filename="$(find raw_description)/urdf/vacuum_gripper/gripper.urdf.xacro" />
+  <!--xacro:include filename="$(find raw_description)/urdf/vacuum_gripper/gripper.urdf.xacro" /-->
+  <!-- schmaltz vacuum gripper -->
+  <xacro:include filename="$(find raw_description)/urdf/schmaltz_gripper/gripper.urdf.xacro" />
+  <!-- arm camera -->
+  <xacro:include filename="$(find raw_description)/urdf/kinect_camera/kinect_camera.urdf.xacro" />
   <!-- sensors -->
   <xacro:include filename="$(find cob_description)/urdf/sensors/sick_s300_laser.urdf.xacro"/>
@@ -40,3 +44,6 @@
     <origin xyz="${gripper_x} ${gripper_y} ${gripper_z}" rpy="${gripper_roll} ${gripper_pitch} ${gripper_yaw}" />
   </xacro:vacuum_gripper>
+  <xacro:kinect_camera name="arm_camera" ros_topic="arm_kinect_camera" parent="gripper_coupling_link" update_rate="30" data_skip="9">
+    <origin xyz="${arm_camera_x} ${arm_camera_y} ${arm_camera_z}" rpy="${arm_camera_roll} ${arm_camera_pitch} ${arm_camera_yaw}" />
+  </xacro:kinect_camera>
 </robot>

Commit message: udate after karlsrhe

File: cob_hardware_config/robots/cob4-7/urdf/calibration_default.urdf.xacro (robot description, xacro)
@@ -116,9 +116,16 @@
 	<xacro:property name="def_head_cam_yaw" value="0.0"/>
         <!-- cam | handeye calibration | relative to head_3_link -->
-        <xacro:property name="def_face_cam_x" value="-0.18486"/>
+        <!--xacro:property name="def_face_cam_x" value="-0.18486"/>
         <xacro:property name="def_face_cam_y" value="0.0"/>
         <xacro:property name="def_face_cam_z" value="0.38953"/>
-        <xacro:property name="def_face_cam_roll" value="0.0"/> <!-- -1.57079 -->
-        <xacro:property name="def_face_cam_pitch" value="-0.1745"/>
-        <xacro:property name="def_face_cam_yaw" value="0.0"/>
+        <xacro:property name="def_face_cam_roll" value="0.0"/--> <!-- -1.57079 -->
+        <!--xacro:property name="def_face_cam_pitch" value="-0.1745"/>
+        <xacro:property name="def_face_cam_yaw" value="0.0"/-->
+	<!-- new ones from ipa_calibration -->
+        <xacro:property name="def_face_cam_x" value="-0.199755"/>
+        <xacro:property name="def_face_cam_y" value="0.0370429"/>
+        <xacro:property name="def_face_cam_z" value="0.358513"/>
+        <xacro:property name="def_face_cam_roll" value="0.0132327"/> <!-- -1.57079 -->
+        <xacro:property name="def_face_cam_pitch" value="-0.121456"/>
+        <xacro:property name="def_face_cam_yaw" value="-0.0432365"/>
 </robot>

Commit message: adapt manual robot arm calibration values

File: cob_hardware_config/robots/cob4-7/urdf/calibration_default.urdf.xacro (robot description, xacro)
@@ -50,6 +50,12 @@
 	<xacro:property name="def_sensorring_yaw" value="0.0"/>
 	<!-- arm right mount positions | relative to torso_3_link -->
+	<!--xacro:property name="def_arm_right_x" value="0.0"/>
+	<xacro:property name="def_arm_right_y" value="-0.014"/>
+	<xacro:property name="def_arm_right_z" value="0.55"/>
+	<xacro:property name="def_arm_right_roll" value="1.57097"/>
+	<xacro:property name="def_arm_right_pitch" value="0"/>
+	<xacro:property name="def_arm_right_yaw" value="0.0"/-->
 	<xacro:property name="def_arm_right_x" value="0.0"/>
-	<xacro:property name="def_arm_right_y" value="-0.014"/>
+	<xacro:property name="def_arm_right_y" value="-0.124"/>
 	<xacro:property name="def_arm_right_z" value="0.55"/>
 	<xacro:property name="def_arm_right_roll" value="1.57097"/>
@@ -57,6 +63,12 @@
 	<xacro:property name="def_arm_right_yaw" value="0.0"/>
 	<!-- arm left mount positions | relative to torso_3_link -->
+	<!--xacro:property name="def_arm_left_x" value="0.0"/>
+	<xacro:property name="def_arm_left_y" value="0.014"/>
+	<xacro:property name="def_arm_left_z" value="0.55"/>
+	<xacro:property name="def_arm_left_roll" value="1.57097"/>
+	<xacro:property name="def_arm_left_pitch" value="0"/>
+	<xacro:property name="def_arm_left_yaw" value="3.14159"/-->
 	<xacro:property name="def_arm_left_x" value="0.0"/>
-	<xacro:property name="def_arm_left_y" value="0.014"/>
+	<xacro:property name="def_arm_left_y" value="0.124"/>
 	<xacro:property name="def_arm_left_z" value="0.55"/>
 	<xacro:property name="def_arm_left_roll" value="1.57097"/>

Commit message: add correct translation and orientation offset values

File: cob_hardware_config/robots/cob4-7/urdf/calibration_default.urdf.xacro (robot description, xacro)
@@ -57,8 +57,8 @@
 	<xacro:property name="def_arm_right_yaw" value="0.0"/-->
 	<xacro:property name="def_arm_right_x" value="0.0"/>
-	<xacro:property name="def_arm_right_y" value="-0.124"/>
+	<xacro:property name="def_arm_right_y" value="-0.1445"/>
 	<xacro:property name="def_arm_right_z" value="0.55"/>
 	<xacro:property name="def_arm_right_roll" value="1.57097"/>
-	<xacro:property name="def_arm_right_pitch" value="0"/>
+	<xacro:property name="def_arm_right_pitch" value="0.78"/>
 	<xacro:property name="def_arm_right_yaw" value="0.0"/>
 	<!-- arm left mount positions | relative to torso_3_link -->
@@ -70,8 +70,8 @@
 	<xacro:property name="def_arm_left_yaw" value="3.14159"/-->
 	<xacro:property name="def_arm_left_x" value="0.0"/>
-	<xacro:property name="def_arm_left_y" value="0.124"/>
+	<xacro:property name="def_arm_left_y" value="0.1445"/>
 	<xacro:property name="def_arm_left_z" value="0.55"/>
 	<xacro:property name="def_arm_left_roll" value="1.57097"/>
-	<xacro:property name="def_arm_left_pitch" value="0"/>
+	<xacro:property name="def_arm_left_pitch" value="-0.78"/>
 	<xacro:property name="def_arm_left_yaw" value="3.14159"/>
         <!-- gripper right mount positions | relative to arm_right_7_link -->
