Commit message: merge stuff from leipzig face cam

File: cob_hardware_config/robots/cob4-7/urdf/cob4-7.urdf.xacro (robot description, xacro)
@@ -58,4 +58,7 @@
     <origin xyz="${head_cam_x} ${head_cam_y} ${head_cam_z}" rpy="${head_cam_roll} ${head_cam_pitch} ${head_cam_yaw}" />
   </xacro:usb_cam>
+  <xacro:realsense name="face_cam" ros_topic="face_cam" parent="head_3_link">
+    <origin xyz="${face_cam_x} ${face_cam_y} ${face_cam_z}" rpy="${face_cam_roll} ${face_cam_pitch} ${face_cam_yaw}" />
+  </xacro:realsense>
   <xacro:cob4_arm name="arm_right" parent="torso_3_link" has_podest="false">
     <origin xyz="${arm_right_x} ${arm_right_y} ${arm_right_z}" rpy="${arm_right_roll} ${arm_right_pitch} ${arm_right_yaw}" />

File: cob_hardware_config/robots/cob4-7/urdf/properties.urdf.xacro (robot description, xacro)
@@ -105,3 +105,10 @@
 	<xacro:property name="head_cam_pitch" value="${def_head_cam_pitch+offset_head_cam_pitch}"/>
 	<xacro:property name="head_cam_yaw" value="${def_head_cam_yaw+offset_head_cam_yaw}"/>
+        <!-- cam | handeye calibration | relative to head_3_link -->
+        <xacro:property name="face_cam_x" value="${def_face_cam_x+offset_face_cam_x}"/>
+        <xacro:property name="face_cam_y" value="${def_face_cam_y+offset_face_cam_y}"/>
+        <xacro:property name="face_cam_z" value="${def_face_cam_z+offset_face_cam_z}"/>
+        <xacro:property name="face_cam_roll" value="${def_face_cam_roll+offset_face_cam_roll}"/>
+        <xacro:property name="face_cam_pitch" value="${def_face_cam_pitch+offset_face_cam_pitch}"/>
+        <xacro:property name="face_cam_yaw" value="${def_face_cam_yaw+offset_face_cam_yaw}"/>
 </robot>

Commit message: added grippers to robot-config

File: cob_hardware_config/robots/cob4-7/urdf/cob4-7.urdf.xacro (robot description, xacro)
@@ -70,3 +70,10 @@
     <origin xyz="${sensorring_cam3d_x} ${sensorring_cam3d_y} ${sensorring_cam3d_z}" rpy="${sensorring_cam3d_roll} ${sensorring_cam3d_pitch} ${sensorring_cam3d_yaw}" />
   </xacro:cob_kinect_v0>
+  <!-- grippers -->
+  <xacro:gripper name="gripper_right" parent="arm_right_7_link">
+    <origin xyz="${gripper_right_x} ${gripper_right_y} ${gripper_right_z}" rpy="${gripper_right_roll} ${gripper_right_pitch} ${gripper_right_yaw}" />
+  </xacro:gripper>
+  <xacro:gripper name="gripper_left" parent="arm_left_7_link">
+    <origin xyz="${gripper_left_x} ${gripper_left_y} ${gripper_left_z}" rpy="${gripper_left_roll} ${gripper_left_pitch} ${gripper_left_yaw}" />
+  </xacro:gripper>
 </robot>

Commit message: comment arm right and other unused

File: cob_hardware_config/robots/cob4-7/urdf/cob4-7.urdf.xacro (robot description, xacro)
@@ -41,33 +41,40 @@
   </xacro:torso>
   <!-- left camera -->
-  <xacro:realsense_zr300 name="torso_cam3d_left" ros_topic="torso_cam3d_left" parent="torso_3_link">
+<!--  <xacro:realsense_zr300 name="torso_cam3d_left" ros_topic="torso_cam3d_left" parent="torso_3_link">
     <origin xyz="${torso_cam3d_left_x} ${torso_cam3d_left_y} ${torso_cam3d_left_z}" rpy="${torso_cam3d_left_roll} ${torso_cam3d_left_pitch} ${torso_cam3d_left_yaw}" />
   </xacro:realsense_zr300>
+-->
   <!-- right camera -->
-  <xacro:realsense_zr300 name="torso_cam3d_right" ros_topic="torso_cam3d_right" parent="torso_3_link">
+<!--  <xacro:realsense_zr300 name="torso_cam3d_right" ros_topic="torso_cam3d_right" parent="torso_3_link">
     <origin xyz="${torso_cam3d_right_x} ${torso_cam3d_right_y} ${torso_cam3d_right_z}" rpy="${torso_cam3d_right_roll} ${torso_cam3d_right_pitch} ${torso_cam3d_right_yaw}" />
   </xacro:realsense_zr300>
+-->
   <!-- down camera -->
-  <xacro:realsense name="torso_cam3d_down" ros_topic="torso_cam3d_down" parent="torso_3_link">
+<!-- <xacro:realsense name="torso_cam3d_down" ros_topic="torso_cam3d_down" parent="torso_3_link">
     <origin xyz="${torso_cam3d_down_x} ${torso_cam3d_down_y} ${torso_cam3d_down_z}" rpy="${torso_cam3d_down_roll} ${torso_cam3d_down_pitch} ${torso_cam3d_down_yaw}" />
   </xacro:realsense>
+-->
   <xacro:head name="head" parent="torso_3_link" dof1="false" dof2="false" dof3="false"> <!-- HotFix: set dof* to true when the HW is repaired -->
     <origin xyz="${head_x} ${head_y} ${head_z}" rpy="${head_roll} ${head_pitch} ${head_yaw}" />
   </xacro:head>
-  <xacro:usb_cam name="head_cam" parent="head_3_link" ros_topic="head_cam" update_rate="10" height="960" width="1280" > <!-- get this from config/head_cam.yaml -->
-    <origin xyz="${head_cam_x} ${head_cam_y} ${head_cam_z}" rpy="${head_cam_roll} ${head_cam_pitch} ${head_cam_yaw}" />
+<!--  <xacro:usb_cam name="head_cam" parent="head_3_link" ros_topic="head_cam" update_rate="10" height="960" width="1280" --> <!-- get this from config/head_cam.yaml -->
+<!--    <origin xyz="${head_cam_x} ${head_cam_y} ${head_cam_z}" rpy="${head_cam_roll} ${head_cam_pitch} ${head_cam_yaw}" />
   </xacro:usb_cam>
   <xacro:realsense name="face_cam" ros_topic="face_cam" parent="head_3_link">
     <origin xyz="${face_cam_x} ${face_cam_y} ${face_cam_z}" rpy="${face_cam_roll} ${face_cam_pitch} ${face_cam_yaw}" />
   </xacro:realsense>
+  -->
+<!--
   <xacro:cob4_arm name="arm_right" parent="torso_3_link" has_podest="false">
     <origin xyz="${arm_right_x} ${arm_right_y} ${arm_right_z}" rpy="${arm_right_roll} ${arm_right_pitch} ${arm_right_yaw}" />
   </xacro:cob4_arm>
+-->
   <xacro:cob4_arm name="arm_left" parent="torso_3_link" has_podest="false">
     <origin xyz="${arm_left_x} ${arm_left_y} ${arm_left_z}" rpy="${arm_left_roll} ${arm_left_pitch} ${arm_left_yaw}" />
   </xacro:cob4_arm>
-  <xacro:gripper name="gripper_right" parent="arm_right_7_link">
+<!--  <xacro:gripper name="gripper_right" parent="arm_right_7_link">
     <origin xyz="${gripper_right_x} ${gripper_right_y} ${gripper_right_z}" rpy="${gripper_right_roll} ${gripper_right_pitch} ${gripper_right_yaw}" />
   </xacro:gripper>
+-->
   <xacro:gripper name="gripper_left" parent="arm_left_7_link">
     <origin xyz="${gripper_left_x} ${gripper_left_y} ${gripper_left_z}" rpy="${gripper_left_roll} ${gripper_left_pitch} ${gripper_left_yaw}" />

Commit message: add arm left on robot

File: cob_hardware_config/robots/cob4-7/urdf/cob4-7.urdf.xacro (robot description, xacro)
@@ -12,5 +12,6 @@
   <xacro:include filename="$(find cob_description)/urdf/cob4_torso/torso.urdf.xacro" />
   <!-- arm -->
-  <xacro:include filename="$(find cob_description)/urdf/cob4_arm/cob4_arm.urdf.xacro" />
+  <!--xacro:include filename="$(find cob_description)/urdf/cob4_arm/cob4_arm.urdf.xacro" /-->
+  <xacro:include filename="$(find cob_description)/urdf/cob4_prob_arm/cob4_prob_arm.urdf.xacro" />
   <!-- hand -->
   <xacro:include filename="$(find cob_description)/urdf/cob4_gripper/gripper.urdf.xacro" />
@@ -58,19 +59,22 @@
     <origin xyz="${head_cam_x} ${head_cam_y} ${head_cam_z}" rpy="${head_cam_roll} ${head_cam_pitch} ${head_cam_yaw}" />
   </xacro:usb_cam>
-  <xacro:realsense name="face_cam" ros_topic="face_cam" parent="head_3_link">
+  <!--xacro:realsense name="face_cam" ros_topic="face_cam" parent="head_3_link">
     <origin xyz="${face_cam_x} ${face_cam_y} ${face_cam_z}" rpy="${face_cam_roll} ${face_cam_pitch} ${face_cam_yaw}" />
-  </xacro:realsense>
-  <xacro:cob4_arm name="arm_right" parent="torso_3_link" has_podest="false">
+  </xacro:realsense-->
+  <!--xacro:cob4_arm name="arm_right" parent="torso_3_link" has_podest="false">
     <origin xyz="${arm_right_x} ${arm_right_y} ${arm_right_z}" rpy="${arm_right_roll} ${arm_right_pitch} ${arm_right_yaw}" />
   </xacro:cob4_arm>
   <xacro:cob4_arm name="arm_left" parent="torso_3_link" has_podest="false">
     <origin xyz="${arm_left_x} ${arm_left_y} ${arm_left_z}" rpy="${arm_left_roll} ${arm_left_pitch} ${arm_left_yaw}" />
-  </xacro:cob4_arm>
-  <xacro:gripper name="gripper_right" parent="arm_right_7_link">
+  </xacro:cob4_arm-->
+  <xacro:cob4_prob_arm name="arm_left" parent="torso_3_link" simulation="false">
+    <origin xyz="${arm_left_x} ${arm_left_y} ${arm_left_z}" rpy="${arm_left_roll} ${arm_left_pitch} ${arm_left_yaw}" />
+  </xacro:cob4_prob_arm>
+  <!--xacro:gripper name="gripper_right" parent="arm_right_7_link">
     <origin xyz="${gripper_right_x} ${gripper_right_y} ${gripper_right_z}" rpy="${gripper_right_roll} ${gripper_right_pitch} ${gripper_right_yaw}" />
   </xacro:gripper>
   <xacro:gripper name="gripper_left" parent="arm_left_7_link">
     <origin xyz="${gripper_left_x} ${gripper_left_y} ${gripper_left_z}" rpy="${gripper_left_roll} ${gripper_left_pitch} ${gripper_left_yaw}" />
-  </xacro:gripper>
+  </xacro:gripper-->
   <xacro:sensorring name="sensorring" parent="head_3_link" active="true">
     <origin xyz="${sensorring_x} ${sensorring_y} ${sensorring_z}" rpy="${sensorring_roll} ${sensorring_pitch} ${sensorring_yaw}" />

Commit message: add left and right arm

File: cob_hardware_config/robots/cob4-7/urdf/cob4-7.urdf.xacro (robot description, xacro)
@@ -68,4 +68,7 @@
     <origin xyz="${arm_left_x} ${arm_left_y} ${arm_left_z}" rpy="${arm_left_roll} ${arm_left_pitch} ${arm_left_yaw}" />
   </xacro:cob4_arm-->
+  <xacro:cob4_prob_arm name="arm_right" parent="torso_3_link" simulation="false">
+    <origin xyz="${arm_right_x} ${arm_right_y} ${arm_right_z}" rpy="${arm_right_roll} ${arm_right_pitch} ${arm_right_yaw}" />
+  </xacro:cob4_prob_arm>
   <xacro:cob4_prob_arm name="arm_left" parent="torso_3_link" simulation="false">
     <origin xyz="${arm_left_x} ${arm_left_y} ${arm_left_z}" rpy="${arm_left_roll} ${arm_left_pitch} ${arm_left_yaw}" />

Commit message: add prob gripper

File: cob_hardware_config/robots/cob4-7/urdf/cob4-7.urdf.xacro (robot description, xacro)
@@ -15,5 +15,6 @@
   <xacro:include filename="$(find cob_description)/urdf/cob4_prob_arm/cob4_prob_arm.urdf.xacro" />
   <!-- hand -->
-  <xacro:include filename="$(find cob_description)/urdf/cob4_gripper/gripper.urdf.xacro" />
+  <!--xacro:include filename="$(find cob_description)/urdf/cob4_gripper/gripper.urdf.xacro" /-->
+  <xacro:include filename="$(find cob_description)/urdf/cob4_prob_gripper/prob_gripper.urdf.xacro" />
   <!-- head -->
   <xacro:include filename="$(find cob_description)/urdf/cob4_head/head.urdf.xacro" />
@@ -80,4 +81,10 @@
     <origin xyz="${gripper_left_x} ${gripper_left_y} ${gripper_left_z}" rpy="${gripper_left_roll} ${gripper_left_pitch} ${gripper_left_yaw}" />
   </xacro:gripper-->
+  <xacro:prob_gripper name="gripper_right" parent="arm_right_gripper_interface_link" orientation="up" simulation="false">
+    <origin xyz="${gripper_right_x} ${gripper_right_y} ${gripper_right_z}" rpy="${gripper_right_roll} ${gripper_right_pitch} ${gripper_right_yaw}" />
+  </xacro:prob_gripper>
+  <xacro:prob_gripper name="gripper_left" parent="arm_left_gripper_interface_link" orientation="up" simulation="false">
+    <origin xyz="${gripper_left_x} ${gripper_left_y} ${gripper_left_z}" rpy="${gripper_left_roll} ${gripper_left_pitch} ${gripper_left_yaw}" />
+  </xacro:prob_gripper>
   <xacro:sensorring name="sensorring" parent="head_3_link" active="${True}">
     <origin xyz="${sensorring_x} ${sensorring_y} ${sensorring_z}" rpy="${sensorring_roll} ${sensorring_pitch} ${sensorring_yaw}" />
