Commit message: add camera3d into joints

File: cob_hardware_config/robots/lwa4p_extended/urdf/lwa4p_extended.urdf.xacro (robot description, xacro)
@@ -7,4 +7,5 @@
   <!-- schunk lwa4p_extended -->
   <xacro:include filename="$(find schunk_description)/urdf/lwa4p_extended/lwa4p_extended.urdf.xacro" />
+  <xacro:include filename="$(find cob_description)/urdf/sensors/kinect.urdf.xacro" />
   <!-- Used for fixing robot to Gazebo -->
   <link name="world"/>
@@ -13,3 +14,6 @@
     <origin xyz="0 0 0.026" rpy="0 0 0" /> <!--slightly above gazebo plane-->
   </xacro:schunk_lwa4p_extended>
+  <xacro:cob_kinect_v0 name="arm_right_cam3d" ros_topic="arm_right_cam3d" parent="arm_2_link" update_rate="30" data_skip="9">
+    <origin xyz="0.08 0 0.0" rpy="-1.57 0 0" />
+  </xacro:cob_kinect_v0>
 </robot>
