Commit message: call both ways of gripper

File: cob_hardware_config/robots/baker/urdf/baker.urdf.xacro (robot description, xacro)
@@ -5,10 +5,14 @@
   <xacro:include filename="$(find cob_description)/urdf/materials.urdf.xacro" />
   <!-- baker_arm -->
-  <xacro:include filename="$(find cob_description)/urdf/baker_arm/baker_arm.urdf.xacro" />
+  <!--xacro:include filename="$(find cob_description)/urdf/baker_arm/baker_arm.urdf.xacro" /-->
   <!-- baker_gripper -->
-  <xacro:include filename="$(find cob_description)/urdf/baker_gripper/baker_gripper.urdf.xacro" />
+   <xacro:include filename="$(find cob_description)/urdf/baker_gripper/baker_gripper.urdf.xacro" />
+  <!--xacro:include filename="$(find cob_description)/urdf/baker_gripper/baker_two_fingure_gripper.urdf.xacro" /-->
   <!-- Used for fixing robot to Gazebo -->
   <link name="world"/>
-  <xacro:baker name="arm" parent="world"/>
-  <xacro:baker_arm_gripper name="gripper" parent="arm_gripper"/>
+  <!--xacro:baker name="arm" parent="world"/-->
+  <xacro:baker_arm_gripper name="gripper" parent="world"/>
+  <!--xacro:baker_gripper prefix="" parent="world">
+    <origin xyz="0.0 0 0.0" rpy="0 0 0"/>
+  </xacro:baker_gripper-->
 </robot>

Commit message: update moveit setup assistance

File: cob_hardware_config/robots/baker/urdf/baker.urdf.xacro (robot description, xacro)
@@ -5,14 +5,14 @@
   <xacro:include filename="$(find cob_description)/urdf/materials.urdf.xacro" />
   <!-- baker_arm -->
-  <!--xacro:include filename="$(find cob_description)/urdf/baker_arm/baker_arm.urdf.xacro" /-->
+  <xacro:include filename="$(find cob_description)/urdf/baker_arm/baker_arm.urdf.xacro" />
   <!-- baker_gripper -->
-   <xacro:include filename="$(find cob_description)/urdf/baker_gripper/baker_gripper.urdf.xacro" />
-  <!--xacro:include filename="$(find cob_description)/urdf/baker_gripper/baker_two_fingure_gripper.urdf.xacro" /-->
+   <!--xacro:include filename="$(find cob_description)/urdf/baker_gripper/baker_gripper.urdf.xacro" /-->
+  <xacro:include filename="$(find cob_description)/urdf/baker_gripper/baker_two_fingure_gripper.urdf.xacro" />
   <!-- Used for fixing robot to Gazebo -->
   <link name="world"/>
-  <!--xacro:baker name="arm" parent="world"/-->
-  <xacro:baker_arm_gripper name="gripper" parent="world"/>
-  <!--xacro:baker_gripper prefix="" parent="world">
-    <origin xyz="0.0 0 0.0" rpy="0 0 0"/>
-  </xacro:baker_gripper-->
+  <xacro:baker name="arm" parent="world"/>
+  <!--xacro:baker_arm_gripper name="gripper" parent="world"/-->
+  <xacro:baker_gripper prefix="" parent="arm_gripper">
+    <origin xyz="0.0 0 0.0" rpy="0 0 -1.57"/>
+  </xacro:baker_gripper>
 </robot>

Commit message: control only one joint

File: cob_hardware_config/robots/baker/urdf/baker.urdf.xacro (robot description, xacro)
@@ -6,13 +6,6 @@
   <!-- baker_arm -->
   <xacro:include filename="$(find cob_description)/urdf/baker_arm/baker_arm.urdf.xacro" />
-  <!-- baker_gripper -->
-   <!--xacro:include filename="$(find cob_description)/urdf/baker_gripper/baker_gripper.urdf.xacro" /-->
-  <xacro:include filename="$(find cob_description)/urdf/baker_gripper/baker_two_fingure_gripper.urdf.xacro" />
   <!-- Used for fixing robot to Gazebo -->
   <link name="world"/>
   <xacro:baker name="arm" parent="world"/>
-  <!--xacro:baker_arm_gripper name="gripper" parent="world"/-->
-  <xacro:baker_gripper prefix="" parent="arm_gripper">
-    <origin xyz="0.0 0 0.0" rpy="0 0 -1.57"/>
-  </xacro:baker_gripper>
 </robot>

Commit message: correct split of can device

File: cob_hardware_config/robots/baker/urdf/baker.urdf.xacro (robot description, xacro)
@@ -5,5 +5,6 @@
   <xacro:include filename="$(find cob_description)/urdf/materials.urdf.xacro" />
   <!-- baker_arm -->
-  <xacro:include filename="$(find cob_description)/urdf/baker_arm/baker_arm.urdf.xacro" />
+  <xacro:include filename="$(find cob_description)/urdf/baker_arm_can0/baker_arm.urdf.xacro" />
+  <xacro:include filename="$(find cob_description)/urdf/baker_arm_can1/baker_arm_can1.urdf.xacro" />
   <!-- baker_gripper -->
    <!--xacro:include filename="$(find cob_description)/urdf/baker_gripper/baker_gripper.urdf.xacro" /-->
@@ -11,8 +12,7 @@
   <!-- Used for fixing robot to Gazebo -->
   <link name="world"/>
-  <xacro:baker name="arm_can0" parent="world"/>
-  <!--xacro:baker_arm_gripper name="gripper" parent="world"/-->
-  <xacro:baker_gripper prefix="" parent="arm_can0_gripper">
-    <origin xyz="0.0 0 0.0" rpy="0 0 -1.57"/>
-  </xacro:baker_gripper>
+  <!-- joint 1 and 2 are in the first CAN bus -->
+  <xacro:baker_arm_can0 name="arm_can0" parent="world"/>
+  <!-- joint 3, 4, 5 are in the second CAN bus-->
+  <xacro:baker_arm_can1 name="arm_can1" parent="arm_can0_link1"/>
 </robot>

Commit message: add gripper and commentout it

File: cob_hardware_config/robots/baker/urdf/baker.urdf.xacro (robot description, xacro)
@@ -9,5 +9,5 @@
   <!-- baker_gripper -->
    <!--xacro:include filename="$(find cob_description)/urdf/baker_gripper/baker_gripper.urdf.xacro" /-->
-  <xacro:include filename="$(find cob_description)/urdf/baker_gripper/baker_two_fingure_gripper.urdf.xacro" />
+  <!--xacro:include filename="$(find cob_description)/urdf/baker_gripper/baker_two_fingure_gripper.urdf.xacro" /-->
   <!-- Used for fixing robot to Gazebo -->
   <link name="world"/>
@@ -16,3 +16,7 @@
   <!-- joint 3, 4, 5 are in the second CAN bus-->
   <xacro:baker_arm_can1 name="arm_can1" parent="arm_can0_link1"/>
+  <!--xacro:baker_arm_gripper name="gripper" parent="world"/-->
+  <!--xacro:baker_gripper prefix="" parent="arm_gripper">
+    <origin xyz="0.0 0 0.0" rpy="0 0 -1.57"/>
+  </xacro:baker_gripper-->
 </robot>
